Commit message: added link 2 and joint 2

File: ros2_ws/src/planar_2r_description/urdf/joints.xacro (robot description, xacro)
@@ -24,3 +24,25 @@
             velocity="2.0"/>
     </joint>
+    <!-- ========================================================= -->
+    <!-- Joint 2                                                   -->
+    <!-- Connects base_link to link1                              -->
+    <!-- ========================================================= -->
+    <joint name="joint2" type="revolute">
+        <parent link="link1"/>
+        <child link="link2"/>
+        <!--
+            The joint 2 starts at the end of link1.
+        -->
+        <origin
+            xyz="${link1_length} 0 0"
+            rpy="0 0 0"/>
+        <!-- Rotation about +Z -->
+        <axis xyz="0 0 1"/>
+        <!-- Joint limits -->
+        <limit
+            lower="-3.14159265"
+            upper="3.14159265"
+            effort="50"
+            velocity="2.0"/>
+    </joint>
 </robot>

File: ros2_ws/src/planar_2r_description/urdf/links.xacro (robot description, xacro)
@@ -92,3 +92,43 @@
         </inertial>
     </link>
+    <!-- ================================================= -->
+    <!-- Link 2                                             -->
+    <!-- Reference frame located at Joint 2                        -->
+    <!-- ================================================= -->
+    <link name="link2">
+        <visual>
+            <origin
+                xyz="${link2_length/2} 0 0"
+                rpy="0 1.57079632679 0"/>
+            <geometry>
+                <cylinder
+                    radius="${link_radius}"
+                    length="${link2_length}"/>
+            </geometry>
+            <material name="link2_material"/>
+        </visual>
+        <collision>
+            <origin
+                xyz="${link2_length/2} 0 0"
+                rpy="0 1.57079632679 0"/>
+            <geometry>
+                <cylinder
+                    radius="${link_radius}"
+                    length="${link2_length}"/>
+            </geometry>
+        </collision>
+        <inertial>
+            <origin
+                xyz="${link2_length/2} 0 0"
+                rpy="0 1.57079632679 0"/>
+            <mass value="1.0"/>
+            <inertia
+                ixx="0.09"
+                ixy="0"
+                ixz="0"
+                iyy="0.09"
+                iyz="0"
+                izz="0.001"/>
+        </inertial>
+    </link>
 </robot>

Commit message: modified and added xacro macros and rviz dfinition and image

File: ros2_ws/src/planar_2r_description/urdf/joints.xacro (robot description, xacro)
@@ -2,47 +2,64 @@
 <robot xmlns:xacro="http://www.ros.org/wiki/xacro">
     <!-- ========================================================= -->
+    <!-- Revolute Joint Macro                                      -->
+    <!-- ========================================================= -->
+    <xacro:macro
+        name="revolute_joint"
+        params="
+            name
+            parent_link
+            child_link
+            xyz
+            rpy
+            axis
+            lower
+            upper
+            effort
+            velocity">
+        <joint name="${name}" type="revolute">
+            <!-- Parent and Child Links -->
+            <parent link="${parent_link}"/>
+            <child link="${child_link}"/>
+            <!-- Joint Frame -->
+            <origin
+                xyz="${xyz}"
+                rpy="${rpy}"/>
+            <!-- Joint Axis -->
+            <axis xyz="${axis}"/>
+            <!-- Joint Limits -->
+            <limit
+                lower="${lower}"
+                upper="${upper}"
+                effort="${effort}"
+                velocity="${velocity}"/>
+        </joint>
+    </xacro:macro>
+    <!-- ========================================================= -->
     <!-- Joint 1                                                   -->
-    <!-- Connects base_link to link1                              -->
     <!-- ========================================================= -->
-    <joint name="joint1" type="revolute">
-        <parent link="base_link"/>
-        <child link="link1"/>
-        <!--
-            The base_link frame is located at Joint 1.
-            Therefore link1 starts exactly at the base frame.
-        -->
-        <origin
-            xyz="0 0 0"
-            rpy="0 0 0"/>
-        <!-- Rotation about +Z -->
-        <axis xyz="0 0 1"/>
-        <!-- Joint limits -->
-        <limit
-            lower="-3.14159265"
-            upper="3.14159265"
-            effort="50"
-            velocity="2.0"/>
-    </joint>
+    <xacro:revolute_joint
+        name="joint1"
+        parent_link="base_link"
+        child_link="link1"
+        xyz="0 0 0"
+        rpy="0 0 0"
+        axis="0 0 1"
+        lower="-3.14159265"
+        upper="3.14159265"
+        effort="50"
+        velocity="2.0"/>
     <!-- ========================================================= -->
     <!-- Joint 2                                                   -->
-    <!-- Connects base_link to link1                              -->
     <!-- ========================================================= -->
-    <joint name="joint2" type="revolute">
-        <parent link="link1"/>
-        <child link="link2"/>
-        <!--
-            The joint 2 starts at the end of link1.
-        -->
-        <origin
-            xyz="${link1_length} 0 0"
-            rpy="0 0 0"/>
-        <!-- Rotation about +Z -->
-        <axis xyz="0 0 1"/>
-        <!-- Joint limits -->
-        <limit
-            lower="-3.14159265"
-            upper="3.14159265"
-            effort="50"
-            velocity="2.0"/>
-    </joint>
+    <xacro:revolute_joint
+        name="joint2"
+        parent_link="link1"
+        child_link="link2"
+        xyz="${link1_length} 0 0"
+        rpy="0 0 0"
+        axis="0 0 1"
+        lower="-3.14159265"
+        upper="3.14159265"
+        effort="50"
+        velocity="2.0"/>
 </robot>

File: ros2_ws/src/planar_2r_description/urdf/links.xacro (robot description, xacro)
@@ -1,24 +1,12 @@
 <?xml version="1.0"?>
 <robot xmlns:xacro="http://www.ros.org/wiki/xacro">
-    <!-- ================================================= -->
-    <!-- Base Link                                          -->
-    <!-- Reference frame located at Joint 1 (top of pedestal)       -->
-    <!-- ================================================= -->
+    <!-- ========================================================= -->
+    <!-- Base Link                                                  -->
+    <!-- ========================================================= -->
     <link name="base_link">
-        <!-- Visual -->
-         <!--
-                Shift the cylinder downward so that the
-                top surface coincides with the base frame.
-            -->
-                <!--
-                  The base_link frame is located at the
-                  top center of the pedestal.
-                  The cylinder is shifted downward by
-                  half its height so that its top surface
-                  coincides with the frame.
-               -->
         <visual>
-            <origin xyz="0 0 ${-base_length/2}"
-                    rpy="0 0 0"/>
+            <origin
+                xyz="0 0 ${-base_length/2}"
+                rpy="0 0 0"/>
             <geometry>
                 <cylinder
@@ -28,8 +16,8 @@
             <material name="base_material"/>
         </visual>
-        <!-- Collision -->
         <collision>
-            <origin xyz="0 0 ${-base_length/2}"
-                    rpy="0 0 0"/>
+            <origin
+                xyz="0 0 ${-base_length/2}"
+                rpy="0 0 0"/>
             <geometry>
                 <cylinder
@@ -38,8 +26,8 @@
             </geometry>
         </collision>
-        <!-- Inertia -->
         <inertial>
-            <origin xyz="0 0 ${-base_length/2}"
-                    rpy="0 0 0"/>
+            <origin
+                xyz="0 0 ${-base_length/2}"
+                rpy="0 0 0"/>
             <mass value="2.0"/>
             <inertia
@@ -52,83 +40,81 @@
         </inertial>
     </link>
-    <!-- ================================================= -->
-    <!-- Link 1                                             -->
-    <!-- Reference frame located at Joint 1                        -->
-    <!-- ================================================= -->
-    <link name="link1">
-        <visual>
-            <origin
-                xyz="${link1_length/2} 0 0"
-                rpy="0 1.57079632679 0"/>
-            <geometry>
-                <cylinder
-                    radius="${link_radius}"
-                    length="${link1_length}"/>
-            </geometry>
-            <material name="link1_material"/>
-        </visual>
-        <collision>
-            <origin
-                xyz="${link1_length/2} 0 0"
-                rpy="0 1.57079632679 0"/>
-            <geometry>
-                <cylinder
-                    radius="${link_radius}"
-                    length="${link1_length}"/>
-            </geometry>
-        </collision>
-        <inertial>
-            <origin
-                xyz="${link1_length/2} 0 0"
-                rpy="0 1.57079632679 0"/>
-            <mass value="1.0"/>
-            <inertia
-                ixx="0.09"
-                ixy="0"
-                ixz="0"
-                iyy="0.09"
-                iyz="0"
-                izz="0.001"/>
-        </inertial>
-    </link>
-    <!-- ================================================= -->
-    <!-- Link 2                                             -->
-    <!-- Reference frame located at Joint 2                        -->
-    <!-- ================================================= -->
-    <link name="link2">
-        <visual>
-            <origin
-                xyz="${link2_length/2} 0 0"
-                rpy="0 1.57079632679 0"/>
-            <geometry>
-                <cylinder
-                    radius="${link_radius}"
-                    length="${link2_length}"/>
-            </geometry>
-            <material name="link2_material"/>
-        </visual>
-        <collision>
-            <origin
-                xyz="${link2_length/2} 0 0"
-                rpy="0 1.57079632679 0"/>
-            <geometry>
-                <cylinder
-                    radius="${link_radius}"
-                    length="${link2_length}"/>
-            </geometry>
-        </collision>
-        <inertial>
-            <origin
-                xyz="${link2_length/2} 0 0"
-                rpy="0 1.57079632679 0"/>
-            <mass value="1.0"/>
-            <inertia
-                ixx="0.09"
-                ixy="0"
-                ixz="0"
-                iyy="0.09"
-                iyz="0"
-                izz="0.001"/>
-        </inertial>
-    </link>
+    <!-- ========================================================= -->
+    <!-- Cylindrical Link Macro                                    -->
+    <!-- ========================================================= -->
+    <xacro:macro
+        name="cylindrical_link"
+        params="
+            name
+            length
+            radius
+            material_name
+            mass
+            ixx
+            iyy
+            izz">
+        <link name="${name}">
+            <!-- Visual -->
+            <visual>
+                <origin
+                    xyz="${length/2} 0 0"
+                    rpy="0 1.57079632679 0"/>
+                <geometry>
+                    <cylinder
+                        radius="${radius}"
+                        length="${length}"/>
+                </geometry>
+                <material name="${material_name}"/>
+            </visual>
+            <!-- Collision -->
+            <collision>
+                <origin
+                    xyz="${length/2} 0 0"
+                    rpy="0 1.57079632679 0"/>
+                <geometry>
+                    <cylinder
+                        radius="${radius}"
+                        length="${length}"/>
+                </geometry>
+            </collision>
+            <!-- Inertia -->
+            <inertial>
+                <origin
+                    xyz="${length/2} 0 0"
+                    rpy="0 1.57079632679 0"/>
+                <mass value="${mass}"/>
+                <inertia
+                    ixx="${ixx}"
+                    ixy="0"
+                    ixz="0"
+                    iyy="${iyy}"
+                    iyz="0"
+                    izz="${izz}"/>
+            </inertial>
+        </link>
+    </xacro:macro>
+    <!-- ========================================================= -->
+    <!-- Link 1                                                    -->
+    <!-- ========================================================= -->
+    <xacro:cylindrical_link
+        name="link1"
+        length="${link1_length}"
+        radius="${link_radius}"
+        material_name="link1_material"
+        mass="1.0"
+        ixx="0.09"
+        iyy="0.09"
+        izz="0.001"/>
+    <!-- ========================================================= -->
+    <!-- Link 2                                                    -->
+    <!-- ========================================================= -->
+    <xacro:cylindrical_link
+        name="link2"
+        length="${link2_length}"
+        radius="${link_radius}"
+        material_name="link2_material"
+        mass="1.0"
+        ixx="0.09"
+        iyy="0.09"
+        izz="0.001"/>
 </robot>

Commit message: the forward kinematics fiest working version using ros 2 node

File: ros2_ws/src/planar_2r_description/urdf/joints.xacro (robot description, xacro)
@@ -36,4 +36,27 @@
     </xacro:macro>
     <!-- ========================================================= -->
+    <!-- Fixed Joint Macro                                         -->
+    <!-- ========================================================= -->
+    <xacro:macro
+        name="fixed_joint"
+        params="
+            name
+            parent_link
+            child_link
+            xyz
+            rpy">
+        <joint
+            name="${name}"
+            type="fixed">
+            <!-- Parent and Child Links -->
+            <parent link="${parent_link}"/>
+            <child link="${child_link}"/>
+            <!-- Joint / Frame Origin -->
+            <origin
+                xyz="${xyz}"
+                rpy="${rpy}"/>
+        </joint>
+    </xacro:macro>
+    <!-- ========================================================= -->
     <!-- Joint 1                                                   -->
     <!-- ========================================================= -->
@@ -63,3 +86,13 @@
         effort="50"
         velocity="2.0"/>
+    <!-- ========================================================= -->
+    <!-- End Effector Fixed Joint                                  -->
+    <!-- Connects link2 to ee_link                                 -->
+    <!-- ========================================================= -->
+    <xacro:fixed_joint
+        name="ee_fixed_joint"
+        parent_link="link2"
+        child_link="ee_link"
+        xyz="${link2_length} 0 0"
+        rpy="0 0 0"/>
 </robot>

File: ros2_ws/src/planar_2r_description/urdf/links.xacro (robot description, xacro)
@@ -95,4 +95,12 @@
     </xacro:macro>
     <!-- ========================================================= -->
+    <!-- End Effector Link Macro                                   -->
+    <!-- ========================================================= -->
+    <xacro:macro
+        name="end_effector_link"
+        params="name">
+        <link name="${name}"/>
+    </xacro:macro>
+    <!-- ========================================================= -->
     <!-- Link 1                                                    -->
     <!-- ========================================================= -->
@@ -118,3 +126,8 @@
         iyy="0.09"
         izz="0.001"/>
+    <!-- ========================================================= -->
+    <!-- End Effector Link                                         -->
+    <!-- ========================================================= -->
+    <xacro:end_effector_link
+        name="ee_link"/>
 </robot>
